File: board_v1/Team1_Wetterstation_EAGLE7.brd (EAGLE design)
At the start: 100 x 80 mm, 47 parts

Commit message: Board Layout v1. Bibliothek hinzugefügt
Parts:
- removed ANEMOMETER: (no value), pinhead:2X04
- removed JP1: (no value), pinhead:1X04
- removed N102: L293E, texas:DIL16
- added J1: RJ11-6X, con-tycoelectronics:RJ11-NO_SHIELD
- added MOTOR: (no value), pinhead:2X06
- added R1, R2: 10k, rcl:R0603
- added WIND: (no value), pinhead:1X02
- moved V100 4.58 mm to (30.5, 63.5), turned to 90 degrees
- turned V102 to 90 degrees
Connections:
- net BLUETOOTH_ON renamed BT_EN
- net N$15 renamed I_CHG
- net N$16 renamed I_BOARD
- net N$17 renamed BAT_STATE
- net N$21 renamed GPS_EN
- removed net GND1: N102.4
- removed net GND2: N102.5
- removed net N$26: ANEMOMETER.3, ANEMOMETER.4
- removed net N$27: ANEMOMETER.5, ANEMOMETER.6
- removed net N$8: JP1.3, N102.11
- removed net N$9: JP1.4, N102.10
- removed net VCC2: N102.8
- new net N$28: J1.4, R2.1, WIND.2
- new net N$29: J1.5, R1.1, WIND.1
- new net N$30: MOTOR.3, MOTOR.4
- new net N$31: MOTOR.1, MOTOR.2
- net +3V3: now also R1.2, R2.2
- net +5V: now also V100.2, V102.2; no longer ANEMOMETER.8, V100.3, V102.3
- net +5VBLUETOOTH: now also V100.3; no longer V100.2
- net 5VGPS: now also V102.3; no longer V102.2
- net GND: now also J1.2, J1.3, MOTOR.5, MOTOR.6; no longer ANEMOMETER.2, N102.12, N102.13
- net N$6: now also MOTOR.11, MOTOR.12; no longer JP1.1, N102.15
- net N$7: now also MOTOR.10, MOTOR.9; no longer JP1.2, N102.14
- net VCCREG: now also MOTOR.7, MOTOR.8; no longer N102.16, N102.9
Routing:
- net GND: track 33.7 -> 402.2 mm
- net +5V: track 200.6 -> 172.6 mm, vias 4 -> 6
- net N$28: track 0.00 -> 16.2 mm
- net N$9: track 10.7 -> 0.00 mm
- net N$8: track 10.7 -> 0.00 mm
- net N$7: track 12.8 -> 2.54 mm
- net N$6: track 12.8 -> 2.54 mm
- net +3V3: track 99.5 -> 109.4 mm, vias 2 -> 3
- net N$29: track 0.00 -> 9.07 mm
- net N$20: track 6.77 -> 12.7 mm, vias 0 -> 2
- net +5VBLUETOOTH: track 31.2 -> 25.3 mm
- net VCCREG: track 108.5 -> 104.4 mm
- net 5VGPS: track 42.7 -> 45.4 mm
- net N$27: track 2.54 -> 0.00 mm
- net N$26: track 2.54 -> 0.00 mm
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- removed copper zone on layer 16, net GND
Other:
- board text added: "12V BAT"
- board text added: "1A"
- board text added: "1B"
- board text added: "2A"
- board text added: "2B"
- board text added: "3V3"
- board text added: "5V"
- board text added: "5VGPS"
- board text added: "BAT_IN"
- board text added: "BAT_STATE"
- board text added: "BT_EN"
- board text added: "CHG_OUT"
- board text added: "EN"
- board text added: "GND"
- board text added: "GPS_EN"
- board text added: "I_BOARD"
- board text added: "I_CHG"
- board text added: "N103"
- board text added: "N104"
- board text added: "RXD"
- board text added: "SPD"
- board text added: "STA"
- board text added: "TXD"
- board text added: "VCC"
- board text added: "VCCREG"
- board text added: "WV"
