File: board_v1/Team1_Wetterstation_EAGLE7.sch (EAGLE design)
At the start: 38 parts, among them IC1 L293E, T1 2N7002BK, T2 2N7002BK, T3 BSS84AKW, T4 BSS84AKW

Commit message: Board Layout v1. Bibliothek hinzugefügt
Parts:
- removed IC1: L293E, texas:L293E
- removed JP1: (no value), pinhead:PINHD-1X4
- removed L1, L2: (no value), rcl:L-US0204/7
- added 12V_BAT, GROUND, VCHARGE, VPANEL: SE14, solpad:SE14
- added 3V3OUT, GPS, WIND: (no value), pinhead:PINHD-1X2
- added 3V3_GND: (no value), pinhead:PINHD-1X6
- added BLUETOOTH, MOTOR: (no value), pinhead:PINHD-2X6
- added J1: RJ11-6X, con-tycoelectronics:RJ11-6X
- added L100, L101: (no value), rcl:L-EU0207/5V
- added R100, R101: (no value), rcl:R-EU_R0603
- R1, R2: value (none) -> 10k
- renumbered C1 to C104, C2 to C105, C3 to C106, C4 to C103, C5 to C101, C6 to C107, C7 to C102, C8 to C100, R3 to R111, R4 to R102, R5 to R103, R6 to R104, R7 to R112, R8 to R113, T1 to V101, T2 to V103, T3 to V100, T4 to V102, U$1 to N103, U$2 to N104
Connections:
- net BATSTATE_PIN? renamed BAT_STATE
- net BLUETOOTH_ON renamed BT_EN
- net N$15 renamed I_CHG
- net N$16 renamed I_BOARD
- net N$21 renamed GPS_EN
- removed net N$17: R105.1
- removed net N$8: IC1.3Y, JP1.3
- removed net N$9: IC1.3A, JP1.4
- removed net VCC: C100.1, C103.1, N100.IN+, N100.IN-, N103.RUN, N103.VIN, N104.RUN, N104.VIN
- new net N$22: BLUETOOTH.1, BLUETOOTH.2
- new net N$23: BLUETOOTH.11, BLUETOOTH.12
- new net N$24: BLUETOOTH.10, BLUETOOTH.9
- new net N$25: BLUETOOTH.7, BLUETOOTH.8
- new net N$28: J1.4, R2.1, WIND.2
- new net N$29: J1.5, R1.1, WIND.1
- new net N$30: MOTOR.3, MOTOR.4
- new net N$31: MOTOR.1, MOTOR.2
- new net VCHARGE: N100.IN-, VCHARGE.MP
- new net VPANEL: N100.IN+, VPANEL.MP
- net +3V3: now also 3V3OUT.1, 3V3_GND.1, 3V3_GND.2, 3V3_GND.3, L100.2, R100.2, R2.2; no longer L2.2
- net +5V: now also L101.2, V100.S, V102.S; no longer L1.2, V100.D, V102.D
- net +5VBLUETOOTH: now also BLUETOOTH.3, V100.D; no longer V100.S
- net 12VBAT: now also 12V_BAT.MP
- net 5VGPS: now also GPS.1, V102.D; no longer V102.S
- net GND: now also 3V3OUT.2, 3V3_GND.4, 3V3_GND.5, 3V3_GND.6, BLUETOOTH.5, GPS.2, GROUND.MP, J1.2, J1.3, MOTOR.5, MOTOR.6, R101.1; no longer IC1.GND3, IC1.GND4, R2.1
- net N$10: now also L101.1, N104.SW; no longer L2.1, N103.SW
- net N$11: now also R100.1, R101.2; no longer R1.1, R2.2
- net N$4: now also R105.1
- net N$5: now also L100.1, N103.SW; no longer L1.1, N104.SW
- net N$6: now also MOTOR.11, MOTOR.12; no longer IC1.4A, JP1.1
- net N$7: now also MOTOR.10, MOTOR.9; no longer IC1.4Y, JP1.2
- net VCCREG: now also C100.1, C103.1, MOTOR.7, MOTOR.8, N103.RUN, N103.VIN, N104.RUN, N104.VIN; no longer IC1.3-4EN, IC1.VCC1
Other:
- note removed: "VBat"
- note removed: "VCharger"
- note removed: "VPanel"
- note removed: "VRegulators"
- moved on the sheet: BAT_STATE, R1, R2
